Commit message: Added 25 joint model (extra joint for hand orientation)

File: shadow_hand/URDF/shadow_hand_left.urdf (robot description, URDF)
Before this commit: robot shadow_left, 33 links, 32 joints
Links:
- link ffdistal: geometry collision mesh filename=meshes/collision/f_distal_pst.stl scale=0.001 0.001 0.001; visual mesh filename=meshes/visual/f_distal_pst.stl scale=0.001 0.001 0.001
- link ffknuckle: geometry collision mesh filename=meshes/collision/f_knuckle_E3M5.stl; visual mesh filename=meshes/visual/f_knuckle_E3M5.stl scale=0.001 0.001 0.001
- link ffmiddle: geometry collision cylinder length=0.025 radius=0.007; collision sphere radius=0.007
- link ffproximal: geometry collision cylinder length=0.040 radius=0.007; visual mesh filename=meshes/visual/f_proximal_E3M5.stl scale=0.001 0.001 0.001
- link forearm: geometry collision box size=0.07 0.07 0.07; collision mesh filename=meshes/collision/forearm_E3M5.stl scale=0.001 0.001 0.001
- link lfdistal: geometry collision mesh filename=meshes/visual/f_distal_pst.stl scale=0.001 0.001 0.001; visual mesh filename=meshes/visual/f_distal_pst.stl scale=0.001 0.001 0.001
- link lfknuckle: geometry collision mesh filename=meshes/collision/f_knuckle_E3M5.stl; visual mesh filename=meshes/visual/f_knuckle_E3M5.stl scale=0.001 0.001 0.001
- link lfmetacarpal: geometry collision box size=0.018 0.024 0.040; visual mesh filename=meshes/visual/lf_metacarpal_E3M5_left.stl scale=0.001 0.001 0.001
- link lfmiddle: geometry collision cylinder length=0.025 radius=0.007; collision sphere radius=0.007
- link lfproximal: geometry collision cylinder length=0.040 radius=0.007; visual mesh filename=meshes/visual/f_proximal_E3M5.stl scale=0.001 0.001 0.001
- link mfdistal: geometry collision mesh filename=meshes/collision/f_distal_pst.stl scale=0.001 0.001 0.001; visual mesh filename=meshes/visual/f_distal_pst.stl scale=0.001 0.001 0.001
- link mfknuckle: geometry collision mesh filename=meshes/collision/f_knuckle_E3M5.stl; visual mesh filename=meshes/visual/f_knuckle_E3M5.stl scale=0.001 0.001 0.001
- link mfmiddle: geometry collision cylinder length=0.025 radius=0.007; collision sphere radius=0.007
- link mfproximal: geometry collision cylinder length=0.040 radius=0.007; visual mesh filename=meshes/visual/f_proximal_E3M5.stl scale=0.001 0.001 0.001
- link palm: geometry collision box size=0.018 0.024 0.004; collision box size=0.020 0.024 0.032
- link rfdistal: geometry collision mesh filename=meshes/collision/f_distal_pst.stl scale=0.001 0.001 0.001; visual mesh filename=meshes/visual/f_distal_pst.stl scale=0.001 0.001 0.001
- link rfknuckle: geometry collision mesh filename=meshes/collision/f_knuckle_E3M5.stl; visual mesh filename=meshes/visual/f_knuckle_E3M5.stl scale=0.001 0.001 0.001
- link rfmiddle: geometry collision cylinder length=0.025 radius=0.007; collision sphere radius=0.007
- link rfproximal: geometry collision cylinder length=0.040 radius=0.007; visual mesh filename=meshes/visual/f_proximal_E3M5.stl scale=0.001 0.001 0.001
- link thdistal: geometry collision mesh filename=meshes/visual/th_distal_pst.stl scale=0.001 0.001 0.001; visual mesh filename=meshes/visual/th_distal_pst.stl scale=0.001 0.001 0.001
- link thmiddle: geometry collision mesh filename=meshes/collision/th_middle_E3M5.stl scale=0.001 0.001 0.001; visual mesh filename=meshes/visual/th_middle_E3M5.stl scale=0.001 0.001 0.001
- link thproximal: geometry collision mesh filename=meshes/collision/th_proximal_E3M5.stl scale=0.001 0.001 0.001; visual mesh filename=meshes/visual/th_proximal_E3M5.stl scale=0.001 0.001 0.001
- link wrist: geometry collision box size=0.027 0.018 0.010; collision box size=0.027 0.018 0.010

File: shadow_hand/URDF/shadow_hand_right_extra_joint.urdf (robot description, URDF)
Before this commit: robot shadow_right, 33 links, 32 joints
Joints:
- removed joint world_joint
- added joint ARMJ1: type revolute, parent world, child forearm, origin xyz=0 -0.010 0.21301 rpy=0 0 1.57079, axis 0 0 1, limit lower=-3.1416 upper=3.1416 effort=10 velocity=2.0
