Commit message: Updated files to use 25df models, added demo

File: shadow_hand/URDF/shadow_hand_left_25df.urdf (robot description, URDF)
Before this commit: robot shadow_right, 33 links, 32 joints
Links:
- link ffdistal: geometry collision mesh filename=meshes/collision/f_distal_pst.stl scale=0.001 0.001 0.001; visual mesh filename=meshes/visual/f_distal_pst.stl scale=0.001 0.001 0.001
- link lfdistal: geometry collision mesh filename=meshes/visual/f_distal_pst.stl scale=0.001 0.001 0.001; visual mesh filename=meshes/visual/f_distal_pst.stl scale=0.001 0.001 0.001
- link lfmetacarpal: geometry collision box size=0.018 0.024 0.040; visual mesh filename=meshes/visual/lf_metacarpal_E3M5_left.stl scale=0.001 0.001 0.001
- link palm: geometry collision box size=0.018 0.024 0.004; collision box size=0.020 0.024 0.032
Joints:
- joint ARMJ1: origin xyz=0 -0.010 0.21301 rpy=0 0 1.57079 -> xyz=0 0 0 rpy=0 0 1.57079
- joint FFJ4: axis 0 -1 0 -> 0 1 0; origin xyz=0.033 0 0.095 rpy=0 0 0 -> xyz=-0.033 0 0.095 rpy=0 0 0
- joint LFJ4: axis 0 1 0 -> 0 -1 0; origin xyz=0.05397275 0 0.03779463 rpy=0 0.9599 0 -> xyz=-0.05397275 0 0.03779463 rpy=0 -0.9599 0
- joint LFJ5: origin xyz=-0.033 0 0.02071 rpy=0 -0.9599 0 -> xyz=0.033 0 0.02071 rpy=0 0.9599 0
- joint MFJ4: axis 0 -1 0 -> 0 1 0; origin xyz=0.011 0 0.099 rpy=0 0 0 -> xyz=-0.011 0 0.099 rpy=0 0 0
- joint RFJ4: axis 0 1 0 -> 0 -1 0; origin xyz=-0.011 0 0.095 rpy=0 0 0 -> xyz=0.011 0 0.095 rpy=0 0 0
- joint THJ3: axis 0 1 0 -> 0 -1 0
- joint THJ4: axis 0 1 0 -> 0 -1 0
- joint THJ5: axis 0 0 -1 -> 0 0 1; origin xyz=0.034 -0.00858 0.029 rpy=-0.785398163397 0 -1.57079632679 -> xyz=-0.034 -0.00858 0.029 rpy=-0.785398163397 0 1.57079632679
- joint WRJ2: axis 0 1 0 -> 0 -1 0
- joint ee_fixed_joint: origin xyz=0.0 0.0 0.0 rpy=0.0 0.0 -1.57079 -> xyz=0.0 0.0 0.00 rpy=0.0 0.0 0.0

Commit message: Letter j in progress

File: shadow_hand/URDF/shadow_hand_left_25df.urdf (robot description, URDF)
Before this commit: robot shadow_left, 33 links, 32 joints
Joints:
- joint WRJ1: limit lower=-0.698131700798 upper=0.488692190558 effort=30 velocity=2.0 -> lower=-1.5708 upper=1.5708 effort=30 velocity=2.0
- joint WRJ2: limit lower=-0.523598775598 upper=0.174532925199 effort=10 velocity=2.0 -> lower=-1.5708 upper=1.5708 effort=10 velocity=2.0

File: shadow_hand/URDF/shadow_hand_right_25df.urdf (robot description, URDF)
Before this commit: robot shadow_right, 33 links, 32 joints
Joints:
- joint WRJ1: limit lower=-0.698131700798 upper=0.488692190558 effort=30 velocity=2.0 -> lower=-1.5708 upper=1.5708 effort=30 velocity=2.0
- joint WRJ2: limit lower=-0.523598775598 upper=0.174532925199 effort=10 velocity=2.0 -> lower=-1.5708 upper=1.5708 effort=10 velocity=2.0
