Commit message: Started to work on extra prismatic joint for sliding repeated letters

File: shadow_hand/URDF/shadow_hand_right_26df.urdf (robot description, URDF)
Before this commit: robot shadow_right, 34 links, 33 joints
Links:
- removed link thdummy
- added link world2
Joints:
- removed joint THJ6
- added joint ARMJ2: type prismatic, parent world2, child world, origin xyz=0 0 0 rpy=0 0 0, axis 0 1 0, limit lower=-0.2 upper=0.2 effort=10 velocity=2.0
- joint THJ4: parent thdummy -> thbase
- joint THJ5: axis 1 0 0 -> 0 0 -1; child thdummy -> thbase; origin xyz=0 0 0 rpy=0 0 0 -> xyz=0.034 -0.00858 0.029 rpy=-0.785398163397 0 -1.57079632679; parent thbase -> palm
- joint WRJ1: limit lower=-0.698131700798 upper=0.488692190558 effort=30 velocity=2.0 -> lower=-1.5708 upper=1.5708 effort=30 velocity=2.0
- joint WRJ2: limit lower=-0.523598775598 upper=0.174532925199 effort=10 velocity=2.0 -> lower=-1.5708 upper=1.5708 effort=10 velocity=2.0
